File: MicroViewUSB.sch (EAGLE design)
At the start: 28 parts, among them J1 MICROVIEW-16ND, Q1 2N7002PW, U1 FT231XS

Commit message: v02 from SparkFun
Other:
- note added: "v02"
- note removed: "v01"
Changed lines of the file:
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@@
 <sheet>
 <plain>
-<text x="240.03" y="6.858" size="3.048" layer="94">v01</text>
+<text x="240.03" y="6.858" size="3.048" layer="94">v02</text>
 <text x="150.622" y="6.858" size="3.048" layer="94">Jim Lindblom, JP Liew, Marchus Schappi</text>
 </plain>
